Commit message: Gazebo Visualization

File: urdf/sbr.urdf (robot description, URDF)
Before this commit: robot SBR, 4 links, 3 joints
Links:
- link base_link: mass None -> 1.0; geometry collision mesh filename=file:///$(find sbr_pjt)/meshes/base_link.STL; visual mesh filename=file:///$(find sbr_pjt)/meshes/base_link.STL
- link left_wheel: mass None -> 1.0; geometry collision mesh filename=file:///$(find sbr_pjt)/meshes/left_wheel.STL; visual mesh filename=file:///$(find sbr_pjt)/meshes/left_wheel.STL
- link right_wheel: mass None -> 1.0; geometry collision mesh filename=file:///$(find sbr_pjt)/meshes/right_wheel.STL; visual mesh filename=file:///$(find sbr_pjt)/meshes/right_wheel.STL

Commit message: Added IMU sensor

File: urdf/sbr.urdf (robot description, URDF)
Before this commit: robot SBR, 4 links, 3 joints
Links:
- added link imu_link, mass 0.001; collision sphere radius=0.02; visual sphere radius=0.02
Joints:
- added joint imu_base_link_joint: type fixed, parent base_link, child imu_link, origin xyz=0.01 0 0.41 rpy=0 0 0

Commit message: Tuned the LQR and Stabilized the Robot

File: urdf/sbr.urdf (robot description, URDF)
Before this commit: robot SBR, 5 links, 4 joints
Links:
- link base_link: mass 1.0 -> 22.9471287282447
- link imu_link: mass 0.001 -> 0.1
- link left_wheel: mass 1.0 -> 3.0
- link right_wheel: mass 1.0 -> 3.0
